File: cmr_link/cmr_link.kicad_pcb (KiCad board)
At the start: 2 copper layers, 0 parts

Commit message: [cmr_link] footprint, net list, layout
Parts:
- added U1: DS90CR288A, tssop-56-DGG, F.Cu at (32.0, 29.8)
Changed lines of the file:
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@@
     (links 0)
     (no_connects 0)
-    (area 0 0 0 0)
+    (area 24.114646 24.817146 39.893354 34.745854)
     (thickness 1.6)
     (drawings 0)
     (tracks 0)
     (zones 0)
-    (modules 0)
+    (modules 1)
     (nets 1)
   )
@@
     (add_net "")
   )
+  (module tssop-56-DGG (layer F.Cu)
+    (at 32.004 29.7815)
+    (fp_text reference U1 (at 0 1.016) (layer F.SilkS)
+      (effects (font (size 1 1) (thickness 0.15)))
+    )
+    (fp_text value DS90CR288A (at 0 -1.016) (layer F.SilkS)
+      (effects (font (size 1 1) (thickness 0.15)))
+    )
+    (fp_arc (start -7 3.05) (end -7 1.5) (angle 90) (layer F.SilkS) (width 0.15))
+    (fp_arc (start -7 3.05) (end -7 1.75) (angle 90) (layer F.SilkS) (width 0.15))
+    (fp_arc (start -7 3.05) (end -7 1.1) (angle 90) (layer F.SilkS) (width 0.15))
+    (fp_line (start -7 -3.05) (end -7 3.05) (layer F.SilkS) (width 0.15))
+    (fp_line (start -7 3.05) (end 7 3.05) (layer F.SilkS) (width 0.15))
+    (fp_line (start 7 3.05) (end 7 -3.05) (layer F.SilkS) (width 0.15))
+    (fp_line (start 7 -3.05) (end -7 -3.05) (layer F.SilkS) (width 0.15))
+    (pad 55 smd rect (at -6.25 -3.825) (size 0.27 1.75)
+      (layers F.Cu F.Paste F.Mask)
+    )
+    (pad 56 smd rect (at -6.75 -3.825) (size 0.27 1.75)
+      (layers F.Cu F.Paste F.Mask)
+    )
+    (pad 54 smd rect (at -5.75 -3.825) (size 0.27 1.75)
+      (layers F.Cu F.Paste F.Mask)
+    )
+    (pad 53 smd rect (at -5.25 -3.825) (size 0.27 1.75)
+      (layers F.Cu F.Paste F.Mask)
+    )
+    (pad 49 smd rect (at -3.25 -3.825) (size 0.27 1.75)
+      (layers F.Cu F.Paste F.Mask)
+    )
+    (pad 50 smd rect (at -3.75 -3.825) (size 0.27 1.75)
+      (layers F.Cu F.Paste F.Mask)
+    )
+    (pad 52 smd rect (at -4.75 -3.825) (size 0.27 1.75)
+      (layers F.Cu F.Paste F.Mask)
+    )
+    (pad 51 smd rect (at -4.25 -3.825) (size 0.27 1.75)
+      (layers F.Cu F.Paste F.Mask)
+    )
+    (pad 43 smd rect (at -0.25 -3.825) (size 0.27 1.75)
+      (layers F.Cu F.Paste F.Mask)
+    )
+    (pad 44 smd rect (at -0.75 -3.825) (size 0.27 1.75)
+      (layers F.Cu F.Paste F.Mask)
+    )
+    (pad 42 smd rect (at 0.25 -3.825) (size 0.27 1.75)
+      (layers F.Cu F.Paste F.Mask)
+    )
+    (pad 41 smd rect (at 0.75 -3.825) (size 0.27 1.75)
+      (layers F.Cu F.Paste F.Mask)
+    )
+    (pad 45 smd rect (at -1.25 -3.825) (size 0.27 1.75)
+      (layers F.Cu F.Paste F.Mask)
+    )
+    (pad 46 smd rect (at -1.75 -3.825) (size 0.27 1.75)
+      (layers F.Cu F.Paste F.Mask)
+    )
+    (pad 48 smd rect (at -2.75 -3.825) (size 0.27 1.75)
+      (layers F.Cu F.Paste F.Mask)
+    )
+    (pad 47 smd rect (at -2.25 -3.825) (size 0.27 1.75)
+      (layers F.Cu F.Paste F.Mask)
+    )
+    (pad 31 smd rect (at 5.75 -3.825) (size 0.27 1.75)
+      (layers F.Cu F.Paste F.Mask)
+    )
+    (pad 32 smd rect (at 5.25 -3.825) (size 0.27 1.75)
+      (layers F.Cu F.Paste F.Mask)
+    )
+    (pad 30 smd rect (at 6.25 -3.825) (size 0.27 1.75)
+      (layers F.Cu F.Paste F.Mask)
+    )
+    (pad 29 smd rect (at 6.75 -3.825) (size 0.27 1.75)
+      (layers F.Cu F.Paste F.Mask)
+    )
+    (pad 35 smd rect (at 3.75 -3.825) (size 0.27 1.75)
+      (layers F.Cu F.Paste F.Mask)
+    )
+    (pad 36 smd rect (at 3.25 -3.825) (size 0.27 1.75)
+      (layers F.Cu F.Paste F.Mask)
+    )
+    (pad 34 smd rect (at 4.25 -3.825) (size 0.27 1.75)
+      (layers F.Cu F.Paste F.Mask)
+    )
+    (pad 33 smd rect (at 4.75 -3.825) (size 0.27 1.75)
+      (layers F.Cu F.Paste F.Mask)
+    )
+    (pad 37 smd rect (at 2.75 -3.825) (size 0.27 1.75)
+      (layers F.Cu F.Paste F.Mask)
+    )
+    (pad 38 smd rect (at 2.25 -3.825) (size 0.27 1.75)
+      (layers F.Cu F.Paste F.Mask)
+    )
+    (pad 40 smd rect (at 1.25 -3.825) (size 0.27 1.75)
+      (layers F.Cu F.Paste F.Mask)
+    )
+    (pad 39 smd rect (at 1.75 -3.825) (size 0.27 1.75)
+      (layers F.Cu F.Paste F.Mask)
+    )
+    (pad 18 smd rect (at 1.75 3.825) (size 0.27 1.75)
+      (layers F.Cu F.Paste F.Mask)
+    )
+    (pad 17 smd rect (at 1.25 3.825) (size 0.27 1.75)
+      (layers F.Cu F.Paste F.Mask)
+    )
+    (pad 19 smd rect (at 2.25 3.825) (size 0.27 1.75)
+      (layers F.Cu F.Paste F.Mask)
+    )
+    (pad 20 smd rect (at 2.75 3.825) (size 0.27 1.75)
+      (layers F.Cu F.Paste F.Mask)
+    )
+    (pad 24 smd rect (at 4.75 3.825) (size 0.27 1.75)
+      (layers F.Cu F.Paste F.Mask)
+    )
+    (pad 23 smd rect (at 4.25 3.825) (size 0.27 1.75)
+      (layers F.Cu F.Paste F.Mask)
+    )
+    (pad 21 smd rect (at 3.25 3.825) (size 0.27 1.75)
+      (layers F.Cu F.Paste F.Mask)
+    )
+    (pad 22 smd rect (at 3.75 3.825) (size 0.27 1.75)
+      (layers F.Cu F.Paste F.Mask)
+    )
+    (pad 28 smd rect (at 6.75 3.825) (size 0.27 1.75)
+      (layers F.Cu F.Paste F.Mask)
+    )
+    (pad 27 smd rect (at 6.25 3.825) (size 0.27 1.75)
+      (layers F.Cu F.Paste F.Mask)
+    )
+    (pad 25 smd rect (at 5.25 3.825) (size 0.27 1.75)
+      (layers F.Cu F.Paste F.Mask)
+    )
+    (pad 26 smd rect (at 5.75 3.825) (size 0.27 1.75)
+      (layers F.Cu F.Paste F.Mask)
+    )
+    (pad 10 smd rect (at -2.25 3.825) (size 0.27 1.75)
+      (layers F.Cu F.Paste F.Mask)
+    )
+    (pad 9 smd rect (at -2.75 3.825) (size 0.27 1.75)
+      (layers F.Cu F.Paste F.Mask)
+    )
+    (pad 11 smd rect (at -1.75 3.825) (size 0.27 1.75)
+      (layers F.Cu F.Paste F.Mask)
+    )
+    (pad 12 smd rect (at -1.25 3.825) (size 0.27 1.75)
+      (layers F.Cu F.Paste F.Mask)
+    )
+    (pad 16 smd rect (at 0.75 3.825) (size 0.27 1.75)
+      (layers F.Cu F.Paste F.Mask)
+    )
+    (pad 15 smd rect (at 0.25 3.825) (size 0.27 1.75)
+      (layers F.Cu F.Paste F.Mask)
+    )
+    (pad 13 smd rect (at -0.75 3.825) (size 0.27 1.75)
+      (layers F.Cu F.Paste F.Mask)
+    )
+    (pad 14 smd rect (at -0.25 3.825) (size 0.27 1.75)
+      (layers F.Cu F.Paste F.Mask)
+    )
+    (pad 6 smd rect (at -4.25 3.825) (size 0.27 1.75)
+      (layers F.Cu F.Paste F.Mask)
+    )
+    (pad 5 smd rect (at -4.75 3.825) (size 0.27 1.75)
+      (layers F.Cu F.Paste F.Mask)
+    )
+    (pad 7 smd rect (at -3.75 3.825) (size 0.27 1.75)
+      (layers F.Cu F.Paste F.Mask)
+    )
+    (pad 8 smd rect (at -3.25 3.825) (size 0.27 1.75)
+      (layers F.Cu F.Paste F.Mask)
+    )
+    (pad 4 smd rect (at -5.25 3.825) (size 0.27 1.75)
+      (layers F.Cu F.Paste F.Mask)
+    )
+    (pad 3 smd rect (at -5.75 3.825) (size 0.27 1.75)
+      (layers F.Cu F.Paste F.Mask)
+    )
+    (pad 1 smd rect (at -6.75 3.825) (size 0.27 1.75)
+      (layers F.Cu F.Paste F.Mask)
+    )
+    (pad 2 smd rect (at -6.25 3.825) (size 0.27 1.75)
+      (layers F.Cu F.Paste F.Mask)
+    )
+  )
 )
