File: cmr_link/cmr_link.sch (KiCad schematic (older format))
At the start: 0 parts

Commit message: [cmr_link] decoder
Parts:
- added U?: DS90CR288A, ~, symbol DS90CR288A
Changed lines of the file:
@@
 Comment4 ""
 $EndDescr
+$Comp
+L DS90CR288A U?
+U 1 1 5491E7BC
+P 5550 3200
+F 0 "U?" V 5500 3200 70  0000 C CNN
+F 1 "DS90CR288A" V 5600 3200 70  0000 C CNN
+F 2 "~" H 5550 2950 60  0000 C CNN
+F 3 "~" H 5550 2950 60  0000 C CNN
+	1    5550 3200
+	1    0    0    -1
+$EndComp
 $EndSCHEMATC

Commit message: [cmr_link] footprint, net list, layout
Parts:
- gave numbers to parts that had none: 1
Changed lines of the file:
@@
 Sheet 1 1
 Title ""
-Date "17 dec 2014"
+Date "17 jan 2015"
 Rev ""
 Comp ""
@@
 $EndDescr
 $Comp
-L DS90CR288A U?
+L DS90CR288A U1
 U 1 1 5491E7BC
 P 5550 3200
-F 0 "U?" V 5500 3200 70  0000 C CNN
+F 0 "U1" V 5500 3200 70  0000 C CNN
 F 1 "DS90CR288A" V 5600 3200 70  0000 C CNN
 F 2 "~" H 5550 2950 60  0000 C CNN
