File: designs/dds_power/dds_power.sch (KiCad schematic (older format))
At the start: 0 parts

Commit message: [dds_power] schematics
Parts:
- added K? (x6): CONN_3, symbol CONN_3
- added P? (x7): Vin, symbol CONN_2
- added R?: 0, symbol R
- added R?: R, symbol R
- added RV?: POT, symbol POT
- added U?: QD48T018033, symbol QD48T018033
Connections:
- new net: P?.2 (PM), U?.1 (Vin+)
- new net: R?.2, U?.2 (On/Off)
- new net: P?.1 (P1), R?.1, U?.3 (Vin-)
- new net: K?.3 (P3), K?.3 (P3), K?.3 (P3), K?.3 (P3), K?.3 (P3), K?.3 (P3), U?.4 (Vout1)
- new net: K?.2 (PM), K?.2 (PM), K?.2 (PM), K?.2 (PM), K?.2 (PM), K?.2 (PM), R?.2, U?.5 (RTN)
- new net: RV?.3, U?.6 (TRIM)
- new net: K?.1 (P1), K?.1 (P1), K?.1 (P1), K?.1 (P1), K?.1 (P1), K?.1 (P1), U?.7 (Vout2)
- new net: R?.1, RV?.1, RV?.2
- new net: P?.1 (P1), P?.1 (P1), P?.1 (P1), P?.1 (P1), P?.1 (P1), P?.1 (P1)
- new net: P?.2 (PM), P?.2 (PM), P?.2 (PM), P?.2 (PM), P?.2 (PM), P?.2 (PM)
