File: designs/dds_power/dds_power.sch (KiCad schematic (older format))
At the start: 17 parts

Commit message: [dds_power] net list
Parts:
- K1, K2, K3, K4, K5, K6: renamed from K?; value CONN_3 -> 1.8_3.3
- P2, P3, P4, P5, P6, P7: renamed from P?; value Vin -> 12V
- R2: renamed from R?; value R -> 0
- gave numbers to parts that had none: 4
Changed lines of the file:
@@
 $EndDescr
 $Comp
-L QD48T018033 U?
+L QD48T018033 U1
 U 1 1 556796D6
 P 3250 2600
-F 0 "U?" H 3250 2550 60  0000 C CNN
+F 0 "U1" H 3250 2550 60  0000 C CNN
 F 1 "QD48T018033" H 3250 2850 60  0000 C CNN
 F 2 "" H 3250 2600 60  0000 C CNN
@@
 $EndComp
 $Comp
-L CONN_2 P?
+L CONN_2 P1
 U 1 1 55679718
 P 1450 2550
-F 0 "P?" V 1400 2550 40  0000 C CNN
+F 0 "P1" V 1400 2550 40  0000 C CNN
 F 1 "Vin" V 1500 2550 40  0000 C CNN
 F 2 "" H 1450 2550 60  0000 C CNN
@@
 $EndComp
 $Comp
-L R R?
+L R R1
 U 1 1 55679800
 P 2200 2900
-F 0 "R?" V 2280 2900 40  0000 C CNN
+F 0 "R1" V 2280 2900 40  0000 C CNN
 F 1 "0" V 2207 2901 40  0000 C CNN
 F 2 "" V 2130 2900 30  0000 C CNN
@@
 Connection ~ 2450 2750
 $Comp
-L R R?
+L R R2
 U 1 1 55679B76
 P 4550 2650
-F 0 "R?" V 4630 2650 40  0000 C CNN
-F 1 "R" V 4557 2651 40  0000 C CNN
+F 0 "R2" V 4630 2650 40  0000 C CNN
+F 1 "0" V 4557 2651 40  0000 C CNN
 F 2 "" V 4480 2650 30  0000 C CNN
 F 3 "" H 4550 2650 30  0000 C CNN
@@
 	3950 2550 4300 2550
 $Comp
-L POT RV?
+L POT RV1
 U 1 1 55679BD9
 P 4300 2300
-F 0 "RV?" H 4300 2200 50  0000 C CNN
+F 0 "RV1" H 4300 2200 50  0000 C CNN
 F 1 "POT" H 4300 2300 50  0000 C CNN
 F 2 "" H 4300 2300 60  0000 C CNN
@@
 	4450 2050 4450 2300
 $Comp
-L CONN_2 P?
+L CONN_2 P2
 U 1 1 55679E0F
 P 1450 3600
-F 0 "P?" V 1400 3600 40  0000 C CNN
-F 1 "Vin" V 1500 3600 40  0000 C CNN
+F 0 "P2" V 1400 3600 40  0000 C CNN
+F 1 "12V" V 1500 3600 40  0000 C CNN
 F 2 "" H 1450 3600 60  0000 C CNN
 F 3 "" H 1450 3600 60  0000 C CNN
@@
 $EndComp
 $Comp
-L CONN_2 P?
+L CONN_2 P3
 U 1 1 55679E79
 P 2000 4150
-F 0 "P?" V 1950 4150 40  0000 C CNN
-F 1 "Vin" V 2050 4150 40  0000 C CNN
+F 0 "P3" V 1950 4150 40  0000 C CNN
+F 1 "12V" V 2050 4150 40  0000 C CNN
 F 2 "" H 2000 4150 60  0000 C CNN
 F 3 "" H 2000 4150 60  0000 C CNN
@@
 $EndComp
 $Comp
-L CONN_2 P?
+L CONN_2 P4
 U 1 1 55679EE1
 P 2400 4150
-F 0 "P?" V 2350 4150 40  0000 C CNN
-F 1 "Vin" V 2450 4150 40  0000 C CNN
+F 0 "P4" V 2350 4150 40  0000 C CNN
+F 1 "12V" V 2450 4150 40  0000 C CNN
 F 2 "" H 2400 4150 60  0000 C CNN
 F 3 "" H 2400 4150 60  0000 C CNN
@@
 $EndComp
 $Comp
-L CONN_2 P?
+L CONN_2 P5
 U 1 1 55679F23
 P 2800 4150
-F 0 "P?" V 2750 4150 40  0000 C CNN
-F 1 "Vin" V 2850 4150 40  0000 C CNN
+F 0 "P5" V 2750 4150 40  0000 C CNN
+F 1 "12V" V 2850 4150 40  0000 C CNN
 F 2 "" H 2800 4150 60  0000 C CNN
 F 3 "" H 2800 4150 60  0000 C CNN
@@
 $EndComp
 $Comp
-L CONN_2 P?
+L CONN_2 P6
 U 1 1 55679F53
 P 3200 4150
-F 0 "P?" V 3150 4150 40  0000 C CNN
-F 1 "Vin" V 3250 4150 40  0000 C CNN
+F 0 "P6" V 3150 4150 40  0000 C CNN
+F 1 "12V" V 3250 4150 40  0000 C CNN
 F 2 "" H 3200 4150 60  0000 C CNN
 F 3 "" H 3200 4150 60  0000 C CNN
@@
 $EndComp
 $Comp
-L CONN_2 P?
+L CONN_2 P7
 U 1 1 55679FF5
 P 3600 4150
-F 0 "P?" V 3550 4150 40  0000 C CNN
-F 1 "Vin" V 3650 4150 40  0000 C CNN
+F 0 "P7" V 3550 4150 40  0000 C CNN
+F 1 "12V" V 3650 4150 40  0000 C CNN
 F 2 "" H 3600 4150 60  0000 C CNN
 F 3 "" H 3600 4150 60  0000 C CNN
@@
 Connection ~ 3100 3500
 $Comp
-L CONN_3 K?
+L CONN_3 K1
 U 1 1 5567B186
 P 4550 3000
-F 0 "K?" V 4500 3000 50  0000 C CNN
-F 1 "CONN_3" V 4600 3000 40  0000 C CNN
+F 0 "K1" V 4500 3000 50  0000 C CNN
+F 1 "1.8_3.3" V 4600 3000 40  0000 C CNN
 F 2 "" H 4550 3000 60  0000 C CNN
 F 3 "" H 4550 3000 60  0000 C CNN
@@
 $EndComp
 $Comp
-L CONN_3 K?
+L CONN_3 K2
 U 1 1 5567B301
 P 4550 3400
-F 0 "K?" V 4500 3400 50  0000 C CNN
-F 1 "CONN_3" V 4600 3400 40  0000 C CNN
+F 0 "K2" V 4500 3400 50  0000 C CNN
+F 1 "1.8_3.3" V 4600 3400 40  0000 C CNN
 F 2 "" H 4550 3400 60  0000 C CNN
 F 3 "" H 4550 3400 60  0000 C CNN
@@
 $EndComp
 $Comp
-L CONN_3 K?
+L CONN_3 K3
 U 1 1 5567B363
 P 4550 3800
-F 0 "K?" V 4500 3800 50  0000 C CNN
-F 1 "CONN_3" V 4600 3800 40  0000 C CNN
+F 0 "K3" V 4500 3800 50  0000 C CNN
+F 1 "1.8_3.3" V 4600 3800 40  0000 C CNN
 F 2 "" H 4550 3800 60  0000 C CNN
 F 3 "" H 4550 3800 60  0000 C CNN
@@
 $EndComp
 $Comp
-L CONN_3 K?
+L CONN_3 K4
 U 1 1 5567B3A5
 P 4550 4200
-F 0 "K?" V 4500 4200 50  0000 C CNN
-F 1 "CONN_3" V 4600 4200 40  0000 C CNN
+F 0 "K4" V 4500 4200 50  0000 C CNN
+F 1 "1.8_3.3" V 4600 4200 40  0000 C CNN
 F 2 "" H 4550 4200 60  0000 C CNN
 F 3 "" H 4550 4200 60  0000 C CNN
@@
 $EndComp
 $Comp
-L CONN_3 K?
+L CONN_3 K5
 U 1 1 5567B3F0
 P 4550 4600
-F 0 "K?" V 4500 4600 50  0000 C CNN
-F 1 "CONN_3" V 4600 4600 40  0000 C CNN
+F 0 "K5" V 4500 4600 50  0000 C CNN
+F 1 "1.8_3.3" V 4600 4600 40  0000 C CNN
 F 2 "" H 4550 4600 60  0000 C CNN
 F 3 "" H 4550 4600 60  0000 C CNN
@@
 $EndComp
 $Comp
-L CONN_3 K?
+L CONN_3 K6
 U 1 1 5567B4C8
 P 4550 5000
-F 0 "K?" V 4500 5000 50  0000 C CNN
-F 1 "CONN_3" V 4600 5000 40  0000 C CNN
+F 0 "K6" V 4500 5000 50  0000 C CNN
+F 1 "1.8_3.3" V 4600 5000 40  0000 C CNN
 F 2 "" H 4550 5000 60  0000 C CNN
 F 3 "" H 4550 5000 60  0000 C CNN

Commit message: [dds_power] connectors
Parts:
- U1: footprint (none) -> qd48t018033:qd48t018033
Changed lines of the file:
@@
 LIBS:memory
 LIBS:xilinx
+LIBS:special
 LIBS:microcontrollers
 LIBS:dsp
@@
 LIBS:contrib
 LIBS:valves
-LIBS:qd48t018033
-LIBS:dds_power-cache
+LIBS:cmr_link
+LIBS:cmr_link-cache
 EELAYER 25 0
 EELAYER END
@@
 F 0 "U1" H 3250 2550 60  0000 C CNN
 F 1 "QD48T018033" H 3250 2850 60  0000 C CNN
-F 2 "" H 3250 2600 60  0000 C CNN
+F 2 "qd48t018033:qd48t018033" H 3250 2600 60  0001 C CNN
 F 3 "" H 3250 2600 60  0000 C CNN
 	1    3250 2600
@@
 F 0 "P1" V 1400 2550 40  0000 C CNN
 F 1 "Vin" V 1500 2550 40  0000 C CNN
-F 2 "" H 1450 2550 60  0000 C CNN
+F 2 "" H 1450 2550 60  0001 C CNN
 F 3 "" H 1450 2550 60  0000 C CNN
 	1    1450 2550
@@
 F 0 "R1" V 2280 2900 40  0000 C CNN
 F 1 "0" V 2207 2901 40  0000 C CNN
-F 2 "" V 2130 2900 30  0000 C CNN
+F 2 "" V 2130 2900 30  0001 C CNN
 F 3 "" H 2200 2900 30  0000 C CNN
 	1    2200 2900
@@
 F 0 "R2" V 4630 2650 40  0000 C CNN
 F 1 "0" V 4557 2651 40  0000 C CNN
-F 2 "" V 4480 2650 30  0000 C CNN
+F 2 "" V 4480 2650 30  0001 C CNN
 F 3 "" H 4550 2650 30  0000 C CNN
 	1    4550 2650
@@
 F 0 "RV1" H 4300 2200 50  0000 C CNN
 F 1 "POT" H 4300 2300 50  0000 C CNN
-F 2 "" H 4300 2300 60  0000 C CNN
+F 2 "" H 4300 2300 60  0001 C CNN
 F 3 "" H 4300 2300 60  0000 C CNN
 	1    4300 2300
@@
 F 0 "P2" V 1400 3600 40  0000 C CNN
 F 1 "12V" V 1500 3600 40  0000 C CNN
-F 2 "" H 1450 3600 60  0000 C CNN
+F 2 "" H 1450 3600 60  0001 C CNN
 F 3 "" H 1450 3600 60  0000 C CNN
 	1    1450 3600
@@
 F 0 "P3" V 1950 4150 40  0000 C CNN
 F 1 "12V" V 2050 4150 40  0000 C CNN
-F 2 "" H 2000 4150 60  0000 C CNN
+F 2 "" H 2000 4150 60  0001 C CNN
 F 3 "" H 2000 4150 60  0000 C CNN
 	1    2000 4150
@@
 F 0 "P4" V 2350 4150 40  0000 C CNN
 F 1 "12V" V 2450 4150 40  0000 C CNN
-F 2 "" H 2400 4150 60  0000 C CNN
+F 2 "" H 2400 4150 60  0001 C CNN
 F 3 "" H 2400 4150 60  0000 C CNN
 	1    2400 4150
@@
 F 0 "P5" V 2750 4150 40  0000 C CNN
 F 1 "12V" V 2850 4150 40  0000 C CNN
-F 2 "" H 2800 4150 60  0000 C CNN
+F 2 "" H 2800 4150 60  0001 C CNN
 F 3 "" H 2800 4150 60  0000 C CNN
 	1    2800 4150
@@
 F 0 "P6" V 3150 4150 40  0000 C CNN
 F 1 "12V" V 3250 4150 40  0000 C CNN
-F 2 "" H 3200 4150 60  0000 C CNN
+F 2 "" H 3200 4150 60  0001 C CNN
 F 3 "" H 3200 4150 60  0000 C CNN
 	1    3200 4150
@@
 F 0 "P7" V 3550 4150 40  0000 C CNN
 F 1 "12V" V 3650 4150 40  0000 C CNN
-F 2 "" H 3600 4150 60  0000 C CNN
+F 2 "" H 3600 4150 60  0001 C CNN
 F 3 "" H 3600 4150 60  0000 C CNN
 	1    3600 4150
@@
 F 0 "K1" V 4500 3000 50  0000 C CNN
 F 1 "1.8_3.3" V 4600 3000 40  0000 C CNN
-F 2 "" H 4550 3000 60  0000 C CNN
+F 2 "" H 4550 3000 60  0001 C CNN
 F 3 "" H 4550 3000 60  0000 C CNN
 	1    4550 3000
@@
 F 0 "K2" V 4500 3400 50  0000 C CNN
 F 1 "1.8_3.3" V 4600 3400 40  0000 C CNN
-F 2 "" H 4550 3400 60  0000 C CNN
+F 2 "" H 4550 3400 60  0001 C CNN
 F 3 "" H 4550 3400 60  0000 C CNN
 	1    4550 3400
@@
 F 0 "K3" V 4500 3800 50  0000 C CNN
 F 1 "1.8_3.3" V 4600 3800 40  0000 C CNN
-F 2 "" H 4550 3800 60  0000 C CNN
+F 2 "" H 4550 3800 60  0001 C CNN
 F 3 "" H 4550 3800 60  0000 C CNN
 	1    4550 3800
@@
 F 0 "K4" V 4500 4200 50  0000 C CNN
 F 1 "1.8_3.3" V 4600 4200 40  0000 C CNN
-F 2 "" H 4550 4200 60  0000 C CNN
+F 2 "" H 4550 4200 60  0001 C CNN
 F 3 "" H 4550 4200 60  0000 C CNN
 	1    4550 4200
@@
 F 0 "K5" V 4500 4600 50  0000 C CNN
 F 1 "1.8_3.3" V 4600 4600 40  0000 C CNN
-F 2 "" H 4550 4600 60  0000 C CNN
+F 2 "" H 4550 4600 60  0001 C CNN
 F 3 "" H 4550 4600 60  0000 C CNN
 	1    4550 4600
@@
 F 0 "K6" V 4500 5000 50  0000 C CNN
 F 1 "1.8_3.3" V 4600 5000 40  0000 C CNN
-F 2 "" H 4550 5000 60  0000 C CNN
+F 2 "" H 4550 5000 60  0001 C CNN
 F 3 "" H 4550 5000 60  0000 C CNN
 	1    4550 5000

Commit message: [dds_power] capacitor
Parts:
- added C? (x3): C, symbol C
- added C? (x4): CP, symbol CP
Connections:
- net at P1.2 (PM), U1.1 (Vin+): now also C?.1, C?.2
- net at P1.1 (P1), R1.1, U1.3 (Vin-): now also C?.1, C?.2
- net at K1.3 (P3), K2.3 (P3), K3.3 (P3)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: now also C?.1, C?.1
- net at K1.2 (PM), K2.2 (PM), K3.2 (PM)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: now also C?.1, C?.2, C?.2, C?.2
- net at K1.1 (P1), K2.1 (P1), K3.1 (P1)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: now also C?.1, C?.2
- new net: C?.1, C?.2
Changed lines of the file:
@@
 LIBS:memory
 LIBS:xilinx
-LIBS:special
 LIBS:microcontrollers
 LIBS:dsp
@@
 LIBS:contrib
 LIBS:valves
-LIBS:cmr_link
-LIBS:cmr_link-cache
+LIBS:qd48t018033
+LIBS:dds_power-cache
 EELAYER 25 0
 EELAYER END
@@
 	0    1    1    0
 $EndComp
-Wire Wire Line
-	2550 2450 1800 2450
-Wire Wire Line
-	1800 2650 1850 2650
-Wire Wire Line
-	1850 2650 1850 2750
-Wire Wire Line
-	1850 2750 2550 2750
-Wire Wire Line
-	2550 2600 1950 2600
-Wire Wire Line
-	1950 2600 1950 2900
-Wire Wire Line
-	2450 2900 2450 2750
-Connection ~ 2450 2750
 $Comp
 L R R2
@@
 	0    1    1    0
 $EndComp
-Wire Wire Line
-	3950 2650 4300 2650
-Wire Wire Line
-	3950 2550 4300 2550
 $Comp
 L POT RV1
@@
 	0    1    1    0
 $EndComp
-Wire Wire Line
-	4450 2300 4800 2300
-Wire Wire Line
-	4800 2300 4800 2650
-Wire Wire Line
-	4300 2050 4450 2050
-Wire Wire Line
-	4450 2050 4450 2300
 $Comp
 L CONN_2 P2
@@
 	0    1    1    0
 $EndComp
-Wire Wire Line
-	1800 3700 3700 3700
-Wire Wire Line
-	2100 3700 2100 3800
-Wire Wire Line
-	2500 3700 2500 3800
-Connection ~ 2100 3700
-Wire Wire Line
-	2900 3700 2900 3800
-Connection ~ 2500 3700
-Wire Wire Line
-	3300 3700 3300 3800
-Connection ~ 2900 3700
-Wire Wire Line
-	3700 3700 3700 3800
-Connection ~ 3300 3700
-Wire Wire Line
-	1800 3500 3500 3500
-Wire Wire Line
-	1900 3500 1900 3800
-Wire Wire Line
-	2300 3500 2300 3800
-Connection ~ 1900 3500
-Wire Wire Line
-	2700 3500 2700 3800
-Connection ~ 2300 3500
-Wire Wire Line
-	3100 3500 3100 3800
-Connection ~ 2700 3500
-Wire Wire Line
-	3500 3500 3500 3800
-Connection ~ 3100 3500
 $Comp
 L CONN_3 K1
@@
 	1    0    0    -1
 $EndComp
+$Comp
+L C C?
+U 1 1 55687ADF
+P 2250 2200
+F 0 "C?" H 2250 2300 40  0000 L CNN
+F 1 "C" H 2256 2115 40  0000 L CNN
+F 2 "" H 2288 2050 30  0000 C CNN
+F 3 "" H 2250 2200 60  0000 C CNN
+	1    2250 2200
+	0    1    1    0
+$EndComp
+$Comp
+L C C?
+U 1 1 55687E96
+P 4500 5450
+F 0 "C?" H 4500 5550 40  0000 L CNN
+F 1 "C" H 4506 5365 40  0000 L CNN
+F 2 "" H 4538 5300 30  0000 C CNN
+F 3 "" H 4500 5450 60  0000 C CNN
+	1    4500 5450
+	1    0    0    -1
+$EndComp
+$Comp
+L C C?
+U 1 1 55687EED
+P 4500 5950
+F 0 "C?" H 4500 6050 40  0000 L CNN
+F 1 "C" H 4506 5865 40  0000 L CNN
+F 2 "" H 4538 5800 30  0000 C CNN
+F 3 "" H 4500 5950 60  0000 C CNN
+	1    4500 5950
+	1    0    0    -1
+$EndComp
+$Comp
+L CP C?
+U 1 1 556883ED
+P 4750 5950
+F 0 "C?" H 4800 6050 40  0000 L CNN
+F 1 "CP" H 4800 5850 40  0000 L CNN
+F 2 "" H 4850 5800 30  0000 C CNN
+F 3 "" H 4750 5950 300 0000 C CNN
+	1    4750 5950
+	-1   0    0    1
+$EndComp
+$Comp
+L CP C?
+U 1 1 556883C0
+P 4750 5450
+F 0 "C?" H 4800 5550 40  0000 L CNN
+F 1 "CP" H 4800 5350 40  0000 L CNN
+F 2 "" H 4850 5300 30  0000 C CNN
+F 3 "" H 4750 5450 300 0000 C CNN
+	1    4750 5450
+	1    0    0    -1
+$EndComp
+Wire Wire Line
+	2550 2450 1800 2450
+Wire Wire Line
+	1800 2650 1850 2650
+Wire Wire Line
+	1850 2650 1850 2750
+Wire Wire Line
+	1850 2750 2550 2750
+Wire Wire Line
+	2550 2600 1950 2600
+Wire Wire Line
+	1950 2600 1950 2900
+Connection ~ 2450 2750
+Wire Wire Line
+	3950 2650 4300 2650
+Wire Wire Line
+	3950 2550 4300 2550
+Wire Wire Line
+	4450 2300 4800 2300
+Wire Wire Line
+	4800 2300 4800 2650
+Wire Wire Line
+	4300 2050 4450 2050
+Wire Wire Line
+	4450 2050 4450 2300
+Wire Wire Line
+	1800 3700 3700 3700
+Wire Wire Line
+	2100 3700 2100 3800
+Wire Wire Line
+	2500 3700 2500 3800
+Connection ~ 2100 3700
+Wire Wire Line
+	2900 3700 2900 3800
+Connection ~ 2500 3700
+Wire Wire Line
+	3300 3700 3300 3800
+Connection ~ 2900 3700
+Wire Wire Line
+	3700 3700 3700 3800
+Connection ~ 3300 3700
+Wire Wire Line
+	1800 3500 3500 3500
+Wire Wire Line
+	1900 3500 1900 3800
+Wire Wire Line
+	2300 3500 2300 3800
+Connection ~ 1900 3500
+Wire Wire Line
+	2700 3500 2700 3800
+Connection ~ 2300 3500
+Wire Wire Line
+	3100 3500 3100 3800
+Connection ~ 2700 3500
+Wire Wire Line
+	3500 3500 3500 3800
+Connection ~ 3100 3500
 Wire Wire Line
 	3950 2450 4150 2450
 Wire Wire Line
-	4150 2450 4150 4900
+	4150 2450 4150 6150
 Wire Wire Line
 	4150 2900 4200 2900
@@
 Connection ~ 4150 4500
 Wire Wire Line
-	4100 2650 4100 5000
+	4100 2650 4100 5700
 Wire Wire Line
 	4100 3000 4200 3000
@@
 	3950 2750 4050 2750
 Wire Wire Line
-	4050 2750 4050 5100
+	4050 2750 4050 5250
 Wire Wire Line
 	4050 3100 4200 3100
@@
 	4050 5100 4200 5100
 Connection ~ 4050 4700
+Connection ~ 2450 2200
+Connection ~ 2050 2450
+Connection ~ 2050 2200
+Wire Wire Line
+	4050 5250 4750 5250
+Connection ~ 4050 5100
+Connection ~ 4500 5250
+Wire Wire Line
+	4500 5750 4500 5650
+Wire Wire Line
+	4750 5650 4750 5750
+Wire Wire Line
+	4150 6150 4750 6150
+Connection ~ 4150 4900
+Connection ~ 4500 6150
+Wire Wire Line
+	4100 5700 4750 5700
+Connection ~ 4500 5700
+Connection ~ 4750 5700
+Connection ~ 4100 5000
+$Comp
+L CP C?
+U 1 1 55688DD5
+P 2050 1900
+F 0 "C?" H 2100 2000 40  0000 L CNN
+F 1 "CP" H 2100 1800 40  0000 L CNN
+F 2 "" H 2150 1750 30  0000 C CNN
+F 3 "" H 2050 1900 300 0000 C CNN
+	1    2050 1900
+	-1   0    0    1
+$EndComp
+$Comp
+L CP C?
+U 1 1 556890A2
+P 2450 1900
+F 0 "C?" H 2500 2000 40  0000 L CNN
+F 1 "CP" H 2500 1800 40  0000 L CNN
+F 2 "" H 2550 1750 30  0000 C CNN
+F 3 "" H 2450 1900 300 0000 C CNN
+	1    2450 1900
+	1    0    0    -1
+$EndComp
+Wire Wire Line
+	2450 2100 2450 2900
+Wire Wire Line
+	2050 2100 2050 2450
+Wire Wire Line
+	2450 1700 2050 1700
 $EndSCHEMATC
