File: designs/dds_power/dds_power.kicad_pcb (KiCad board)
At the start: 2 copper layers, 0 parts

Commit message: [dds_power] pcb
Parts:
- added C1: CP, Capacitors_ThroughHole:C_Radial_D5_L11_P2, F.Cu at (137.2, 117.5)
- added C2: C, Capacitors_SMD:C_1206, B.Cu at (141.0, 122.6)
- added C3: CP, Capacitors_ThroughHole:C_Radial_D5_L11_P2, F.Cu at (144.8, 117.5)
- added C4: C, Capacitors_SMD:C_1206, B.Cu at (181.0, 107.3)
- added C5: C, Capacitors_SMD:C_1206, B.Cu at (181.0, 118.1)
- added C6: CP, Capacitors_ThroughHole:C_Radial_D5_L11_P2, F.Cu at (176.5, 106.7)
- added C7: CP, Capacitors_ThroughHole:C_Radial_D5_L11_P2, F.Cu at (176.5, 118.7)
- added K1: 1.8_3.3, cmr_link:3-pins_150mil, F.Cu at (156.2, 123.2)
- added K2: 1.8_3.3, cmr_link:3-pins_150mil, F.Cu at (167.6, 134.0)
- added K3: 1.8_3.3, cmr_link:3-pins_150mil, F.Cu at (174.6, 98.4)
- added K4: 1.8_3.3, cmr_link:3-pins_150mil, F.Cu at (181.6, 134.0)
- added K5: 1.8_3.3, cmr_link:3-pins_150mil, F.Cu at (156.2, 109.9)
- added K6: 1.8_3.3, cmr_link:3-pins_150mil, F.Cu at (159.4, 98.4)
- added P1: CONN_3, cmr_link:3-pins_150mil, F.Cu at (141.0, 128.3)
- added P2: 12V, cmr_link:2-pins_150mil, F.Cu at (144.8, 147.3)
- added P3: 12V, cmr_link:2-pins_150mil, F.Cu at (177.2, 147.3)
- added P4: 12V, cmr_link:2-pins_150mil, F.Cu at (134.0, 147.3)
- added P5: 12V, cmr_link:2-pins_150mil, F.Cu at (188.0, 147.3)
- added P6: 12V, cmr_link:2-pins_150mil, F.Cu at (155.6, 147.3)
- added P7: 12V, cmr_link:2-pins_150mil, F.Cu at (166.4, 147.3)
- added R1: 0, Resistors_SMD:R_0603, F.Cu at (133.3, 109.2)
- added R2: 0, Resistors_SMD:R_0603, F.Cu at (188.0, 110.5)
- added R3: 0, Resistors_SMD:R_0603, F.Cu at (144.1, 134.6)
- added RV1: POT, Potentiometers:Potentiometer_Bourns_3005_Angular_ScrewFront, B.Cu at (189.9, 106.0)
- added U1: QD48T018033, qd48t018033:qd48t018033, B.Cu at (129.5, 132.1)
Routing:
- net Net-(C4-Pad2): track 0.00 -> 573.6 mm, vias 0 -> 2
- net Net-(C4-Pad1): track 0.00 -> 394.4 mm, vias 0 -> 1
- net Net-(C5-Pad2): track 0.00 -> 389.2 mm, vias 0 -> 1
- net Net-(C2-Pad1): track 0.00 -> 39.6 mm
- net GND: track 0.00 -> 22.9 mm
- net Net-(C1-Pad1): track 0.00 -> 20.5 mm
- net Net-(R2-Pad1): track 0.00 -> 9.93 mm
- net Net-(RV1-Pad3): track 0.00 -> 6.63 mm
- net Net-(C1-Pad2): track 0.00 -> 5.62 mm
- net Net-(R1-Pad2): track 0.00 -> 3.75 mm
- added copper zone on F.Cu, net Net-(C4-Pad1)
- added copper zone on In1.Cu, net Net-(C4-Pad2)
- added copper zone on In2.Cu, net Net-(C5-Pad2)
- added copper zone on B.Cu, net Net-(P2-Pad1)
- added copper zone on In1.Cu, net Net-(P2-Pad1)
- added copper zone on F.Cu, net Net-(P2-Pad2)
- added copper zone on In2.Cu, net Net-(P2-Pad2)
Other:
- board outline added: 64.8 x 57.8 mm
- copper layers 2 -> 4
- net class Normal added: clearance 0.2, trace_width 1, via_dia 0.8, via_drill 0.6
- net class Thick added: clearance 0.2, trace_width 2, via_dia 0.8, via_drill 0.6

Commit message: [dds_power] tweak
Parts:
- K1, K2, K3, K4, K5, K6: value 1.8_3.3 -> 3.3_1.8
- moved P2 5.08 mm to (144.8, 142.2)
- moved P3 5.08 mm to (177.2, 142.2)
- moved P4 5.08 mm to (134.0, 142.2)
- moved P5 5.08 mm to (188.0, 142.2)
- moved P6 5.08 mm to (155.6, 142.2)
- moved P7 5.08 mm to (166.4, 142.2)
Routing:
- net Net-(C2-Pad1): track 39.6 -> 57.1 mm
- added copper zone on F.Cu, net Net-(P2-Pad1)
- added copper zone on In2.Cu, net Net-(P2-Pad1)
- added copper zone on B.Cu, net Net-(P2-Pad2)
- added copper zone on In1.Cu, net Net-(P2-Pad2)
- removed copper zone on B.Cu, net Net-(P2-Pad1)
- removed copper zone on In1.Cu, net Net-(P2-Pad1)
- removed copper zone on F.Cu, net Net-(P2-Pad2)
- removed copper zone on In2.Cu, net Net-(P2-Pad2)
Other:
- board size 64.8 x 57.8 mm -> 64.8 x 52.7 mm
- board text added: "+"
