File: designs/regulator/regulator.kicad_pcb (KiCad board)
At the start: 4 copper layers, 52.5 x 22.5 mm, 34 parts, among them J1 Conn_01x03, J2 Conn_01x03, U1 LT3089-TSSOP, U2 LT3090-MSOP

Commit message: [designs/regulator] Tweak size
Parts:
- moved C1 5.52 mm to (133.6, 104.4)
- moved J1 2.73 mm to (122.9, 101.3)
- moved C2 1.75 mm to (138.9, 95.2)
Routing:
- net GND: track 202.1 -> 429.3 mm, vias 4 -> 57
- net VIN+: track 34.6 -> 37.7 mm
Other:
- board size 52.5 x 22.5 mm -> 56.4 x 20.3 mm
